File: ptm-60nrf.kicad_pcb (KiCad board)
At the start: 2 copper layers, 285 x 94.6 mm, 158 parts, among them J1 USB_C_Receptacle_USB2.0, J2 BAT, J4 SWD, Q1 AO3407, U1 TP4054, U2 XC6220B331MR-G, U3 nRF52840_holyiot_18010, U4 SRV05-4

Commit message: cosmetic adjustments
Routing:
- net COL1: track 313.8 -> 342.1 mm
- net COL11: track 199.5 -> 227.3 mm
- net COL7: track 157.0 -> 183.4 mm
- net COL3: track 252.7 -> 276.1 mm
- net COL9: track 169.1 -> 185.8 mm
- net COL5: track 251.3 -> 267.3 mm
- net COL12: track 197.2 -> 187.6 mm
- net COL2: track 266.0 -> 257.9 mm
- net COL4: track 207.1 -> 200.7 mm
- net COL10: track 136.2 -> 130.4 mm
- net COL8: track 114.2 -> 108.7 mm
- net COL6: track 172.7 -> 178.2 mm
- net GND: vias 22 -> 23
- net (no net): vias 1 -> 0

Commit message: further cosmetic adjustments
Parts:
- moved D32 3.07 mm to (285.4, 37.6), turned to 0 degrees
- moved D37 0.66 mm to (108.0, 71.3)
- moved D39 0.66 mm to (129.5, 71.3)
- moved D38 0.66 mm to (110.5, 71.3)
- moved D45 0.65 mm to (243.8, 71.4)
- moved D44 0.65 mm to (241.3, 71.4)
- moved D46 0.65 mm to (260.2, 71.4)
- moved D35 0.65 mm to (70.0, 71.3)
- moved D40 0.64 mm to (165.2, 71.4)
- moved D42 0.63 mm to (203.2, 71.4)
- moved D36 0.63 mm to (72.4, 71.3)
- moved D41 0.62 mm to (167.7, 71.4)
- moved D43 0.62 mm to (205.8, 71.4)
- moved D33 0.54 mm to (38.0, 71.5)
- moved D64 0.39 mm to (286.3, 75.2)
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Routing:
- net ROW4: track 286.7 -> 271.1 mm
- net ROW2: track 289.0 -> 297.5 mm
- net ROW3: track 275.9 -> 281.4 mm
- net Net-(D32-Pad2): track 12.6 -> 8.86 mm
- net ROW1: track 327.3 -> 328.9 mm
- net COL5: track 267.3 -> 268.8 mm
- net Net-(D37-Pad2): track 15.7 -> 15.0 mm
- net Net-(D44-Pad2): track 15.2 -> 14.6 mm
- net Net-(D38-Pad2): track 20.8 -> 20.1 mm
- net Net-(D42-Pad2): track 15.3 -> 14.7 mm
- net Net-(D35-Pad2): track 16.0 -> 15.3 mm
- net Net-(D39-Pad2): track 21.1 -> 20.5 mm
- net Net-(D46-Pad2): track 25.1 -> 24.5 mm
- net Net-(D45-Pad2): track 20.3 -> 19.7 mm
- net Net-(D41-Pad2): track 21.0 -> 20.4 mm
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
Commit message: further beautification
Routing:
- net COL1: track 342.1 -> 292.8 mm
- net COL3: track 276.1 -> 230.6 mm
- net COL7: track 183.4 -> 141.6 mm
- net COL11: track 227.3 -> 189.1 mm
- net COL5: track 268.8 -> 239.7 mm
- net COL9: track 185.8 -> 160.2 mm
- net COL6: track 178.2 -> 170.0 mm
- net COL13: track 218.2 -> 216.4 mm
- net COL0: track 320.1 -> 318.9 mm
- net COL14: track 190.1 -> 189.1 mm
- net GND: vias 22 -> 21

Commit message: Cosmetic changes
Routing:
- net COL11: track 189.1 -> 205.1 mm
- net COL8: track 109.1 -> 102.5 mm
- net COL4: track 200.9 -> 196.4 mm
- net ROW0: track 336.0 -> 333.6 mm
- net COL12: track 188.0 -> 185.7 mm
- net COL10: track 130.6 -> 128.6 mm
- net ROW1: track 328.9 -> 327.2 mm
- net COL3: track 230.6 -> 232.1 mm
- net COL7: track 141.6 -> 142.8 mm
- net ROW2: track 297.5 -> 296.5 mm
- net COL2: track 258.1 -> 257.2 mm
- net COL1: track 292.8 -> 292.1 mm

Commit message: further improvements
Parts:
- moved D70 26.4 mm to (252.8, 94.0), turned to 270 degrees
- moved D69 16.2 mm to (249.0, 94.0), turned to 270 degrees
- moved D71 14.8 mm to (277.1, 94.0), turned to 270 degrees
Routing:
- net COL14: track 189.1 -> 254.0 mm
- net COL12: track 185.7 -> 213.7 mm, vias 1 -> 2
- net Net-(D69-Pad2): track 18.6 -> 5.34 mm
- net COL11: track 205.1 -> 215.5 mm
- net ROW4: track 271.1 -> 280.4 mm
- net COL13: track 216.4 -> 225.0 mm
- net Net-(D71-Pad2): track 24.0 -> 17.2 mm
- net COL0: track 318.9 -> 314.2 mm
- net Net-(D70-Pad2): track 14.2 -> 17.7 mm
- net VBAT: track 88.0 -> 90.1 mm
- net COL9: track 160.0 -> 159.3 mm
- net ROW3: track 281.4 -> 282.1 mm
- net GND: vias 21 -> 22

Commit message: created branch 0.2 for alternate mcu location. Heavy cleanup
Parts:
- G***: moved to B.Cu
- moved G*** 105.6 mm to (117.9, 100.7), turned to 180 degrees
- moved J4 55.1 mm to (228.4, 106.0)
- moved R6 26.1 mm to (179.8, 100.0), turned to 0 degrees
- moved R7 25.6 mm to (179.8, 101.7), turned to 180 degrees
- moved Reset1 12.6 mm to (176.9, 95.4), turned to 180 degrees
- moved U3 5.78 mm to (200.9, 101.5), turned to 0 degrees
Connections:
- U3 pad 10: COL12 -> COL3
- U3 pad 11: COL13 -> COL4
- U3 pad 12: COL14 -> COL5
- U3 pad 13: COL0 -> COL6
- U3 pad 15: COL1 -> COL7
- U3 pad 16: COL2 -> COL8
- U3 pad 17: COL3 -> ROW3
- U3 pad 18: COL4 -> ROW2
- U3 pad 19: COL5 -> ROW1
- U3 pad 20: COL6 -> ROW0
- U3 pad 28: COL7 -> ROW4
- U3 pad 29: COL8 -> COL9
- U3 pad 30: ROW4 -> COL10
- U3 pad 33: ROW3 -> COL11
- U3 pad 34: ROW2 -> COL12
- U3 pad 35: ROW1 -> COL13
- U3 pad 36: ROW0 -> COL14
- U3 pad 7: COL9 -> COL0
- U3 pad 8: COL10 -> COL1
- U3 pad 9: COL11 -> COL2
Routing:
- net VDD: track 78.7 -> 125.5 mm, vias 1 -> 3
- net VBAT: track 90.1 -> 58.9 mm, vias 4 -> 2
- net GND: track 94.7 -> 73.3 mm, vias 22 -> 25
- net RES: track 15.0 -> 33.6 mm, vias 0 -> 2
- net COL10: track 128.9 -> 110.6 mm
- net COL9: track 159.3 -> 141.6 mm
- net USB-D+: track 210.5 -> 225.7 mm
- net COL6: track 170.0 -> 185.0 mm
- net COL5: track 239.7 -> 253.1 mm
- net COL13: track 225.0 -> 211.6 mm
- net COL8: track 102.5 -> 115.0 mm
- net USB-D-: track 213.0 -> 225.5 mm
- net COL14: track 254.0 -> 241.7 mm
- net COL4: track 196.4 -> 208.5 mm
- net COL7: track 142.8 -> 153.8 mm
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Other:
- outline, holes or cut-outs redrawn
- board text added: "Rev. 0.2"
- board text removed: "Rev. 0.1"

Commit message: updated branch and ordered pcb prototype
Parts:
- C1: value 1µF -> 1nF
- D10, D11, D12, D13, D14, D15, D16, D18, D19, D20, D21, D22, D23, D24, D25, D26, D27, D28, D29, D3, D30, D31, D32, D33, D35, D36, D37, D38, D39, D4, D40, D41, D42, D43, D44, D45, D46, D47, D49, D5, D51, D52, D53, D54, D55, D56, D57, D58, D59, D6, D60, D61, D62, D64, D65, D66, D67, D68, D69, D7, D70, D71, D8, D9: value D_Small -> 1n4148; footprint Diode_SMD:D_0603_1608Metric -> Diode_SMD:D_SOD-323F
- D2: footprint Diode_SMD:D_SOD-123 -> Diode_SMD:D_SMA
- R6: value 820K -> 1M
- moved R3 1.84 mm to (133.1, 95.5)
- moved D2 1.04 mm to (136.1, 96.5)
- moved D52 0.43 mm to (79.2, 75.2)
- moved D53 0.37 mm to (82.0, 75.2)
- moved D69 0.26 mm to (249.0, 94.2)
- moved D70 0.26 mm to (252.8, 94.2)
Routing:
- net Net-(D2-Pad1): track 6.26 -> 7.98 mm
- net ROW3: track 289.3 -> 287.6 mm
- net ROW1: track 327.8 -> 326.1 mm
- net ROW0: track 335.2 -> 333.6 mm
- net ROW2: track 295.5 -> 294.4 mm
- net VBUS: track 269.1 -> 270.1 mm
- net Net-(D70-Pad2): track 17.7 -> 18.5 mm
- net Net-(D49-Pad2): track 13.9 -> 13.3 mm
- net Net-(D51-Pad2): track 12.0 -> 11.4 mm
- net Net-(D69-Pad2): track 5.34 -> 5.90 mm
- net Net-(D52-Pad2): track 7.43 -> 6.88 mm
- net Net-(D53-Pad2): track 12.5 -> 12.0 mm

Commit message: cosmetic improvements of a major degree - v0.3
Parts:
- moved D70 22.4 mm to (274.7, 89.6)
- moved D66 22.2 mm to (59.4, 89.6), turned to 270 degrees
- moved D65 22.0 mm to (35.6, 89.6), turned to 270 degrees
- moved D67 15.8 mm to (83.2, 89.6), turned to 270 degrees
- moved D71 7.88 mm to (283.7, 89.6)
- moved D69 7.64 mm to (255.1, 89.6)
- moved D68 5.78 mm to (164.2, 90.1)
- moved D19 2.57 mm to (29.9, 38.7)
- moved J2 1.49 mm to (151.0, 102.9)
- moved D3 1.22 mm to (29.9, 32.9)
- moved D33 1.09 mm to (39.1, 71.4)
Routing:
- net VBUS: track 270.1 -> 379.0 mm
- net USB-D-: track 225.5 -> 266.0 mm
- net USB-D+: track 225.7 -> 264.8 mm
- net ROW3: track 287.6 -> 274.5 mm
- net Net-(D66-Pad2): track 19.2 -> 7.75 mm
- net Net-(D65-Pad2): track 18.8 -> 7.76 mm
- net Net-(D69-Pad2): track 5.90 -> 16.2 mm
- net ROW4: track 272.3 -> 263.1 mm, vias 4 -> 2
- net GND: track 73.3 -> 64.8 mm, vias 25 -> 24
- net COL14: track 241.7 -> 233.2 mm
- net COL1: track 299.4 -> 292.7 mm
- net Net-(D70-Pad2): track 18.5 -> 12.0 mm
- net COL2: track 266.1 -> 259.7 mm
- net COL12: track 204.9 -> 201.2 mm
- net COL5: track 253.1 -> 249.6 mm
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Other:
- board text added: "Rev. 0.3"
- board text removed: "Rev. 0.2"
