File: ptm-60nrf.kicad_pcb (KiCad board)
At the start: 2 copper layers, 285 x 94.6 mm, 158 parts, among them J1 USB_C_Receptacle_USB2.0, J2 BAT, J4 SWD, Q1 AO3407, U1 TP4054, U2 XC6220B331MR-G, U3 nRF52840_holyiot_18010, U4 SRV05-4

Commit message: improved parts placements and silkscreen text (jlc compatible)
Parts:
- moved R1 5.85 mm to (151.6, 95.8)
- moved R2 5.03 mm to (151.5, 97.9), turned to 180 degrees
- moved U1 3.98 mm to (148.0, 99.0)
- moved J2 2.25 mm to (148.9, 102.2)
- moved G*** 1.77 mm to (116.5, 101.7)
- moved D1 1.27 mm to (147.9, 95.8), turned to 180 degrees
- moved R4 0.40 mm to (41.3, 30.7)
- moved C1 0.39 mm to (147.9, 93.6), turned to 180 degrees
- moved U4 0.26 mm to (37.6, 30.6)
- moved R5 0.23 mm to (33.9, 30.8)
Routing:
- net COL5: track 249.6 -> 208.4 mm
- net GND: track 64.8 -> 82.1 mm, vias 24 -> 23
- net VBUS: track 379.0 -> 366.4 mm
- net VDD: track 125.5 -> 113.7 mm, vias 3 -> 2
- net USB-D-: track 266.0 -> 257.6 mm
- net USB-D+: track 264.8 -> 256.9 mm
- net Net-(R1-Pad2): track 6.20 -> 11.4 mm
- net ROW1: track 328.9 -> 325.2 mm
- net ROW0: track 333.7 -> 330.3 mm
- net ROW2: track 293.1 -> 291.2 mm
- net ROW3: track 274.5 -> 276.1 mm
- net Net-(R2-Pad2): track 2.74 -> 1.77 mm
- net VBAT: track 59.2 -> 58.3 mm, vias 2 -> 1
- net Net-(D1-Pad1): track 2.53 -> 1.92 mm
- net COL6: track 181.8 -> 181.2 mm
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
Commit message: modified to use BAV70 diodes
Parts:
- removed the D18 at (286.9, 33.7)
- removed D38, D39, D40, D41, D42, D43, D44, D45, D46, D47, D49, D51, D52, D53, D54, D55, D56, D57, D58, D59, D60, D61, D62, D64, D65, D66, D68, D69, D70, D71: 1n4148, Diode_SMD:D_SOD-323F
- added D17: BAV70, Package_TO_SOT_SMD:SOT-23, B.Cu at (282.5, 37.9)
- added D33: BAV70, Package_TO_SOT_SMD:SOT-23, B.Cu at (46.0, 90.0)
- D10, D11, D12, D13, D14, D15, D16, D19, D20, D21, D22, D23, D24, D26, D27, D28, D29, D30, D31, D32, D37, D4, D5, D6, D7, D8, D9: value 1n4148 -> BAV70; footprint Diode_SMD:D_SOD-323F -> Package_TO_SOT_SMD:SOT-23
- moved D37 174.5 mm to (281.5, 90.0)
- moved D36 173.8 mm to (245.2, 90.1), turned to 270 degrees
- moved D25 152.3 mm to (293.4, 67.2), turned to 90 degrees
- moved D26 139.0 mm to (45.6, 75.0), turned to 90 degrees
- moved D24 125.3 mm to (261.8, 71.6)
- moved D23 125.1 mm to (226.3, 71.5)
- moved D11 124.9 mm to (47.6, 37.1)
- moved D12 120.6 mm to (87.5, 37.1)
- moved D10 116.7 mm to (286.7, 33.7), turned to 270 degrees
- moved D9 114.2 mm to (248.6, 33.7), turned to 270 degrees
- moved D27 106.0 mm to (83.1, 75.0), turned to 90 degrees
- moved D28 103.4 mm to (121.2, 75.0), turned to 90 degrees
- moved D35 96.1 mm to (164.2, 90.1), turned to 270 degrees
- moved D22 89.0 mm to (185.3, 71.5)
- moved D21 86.5 mm to (147.2, 71.5)
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- renumbered D33 to D18, D67 to D34
Connections:
- D10 pad 1: ROW0 -> Net-(D10-Pad1)
- D11 pad 1: ROW0 -> Net-(D11-Pad1)
- D12 pad 1: ROW0 -> Net-(D12-Pad1)
- D13 pad 1: ROW0 -> Net-(D13-Pad1)
- D14 pad 1: ROW0 -> Net-(D14-Pad1)
- D15 pad 1: ROW0 -> Net-(D15-Pad1)
- D16 pad 1: ROW0 -> Net-(D16-Pad1)
- D19 pad 1: ROW1 -> Net-(D19-Pad1)
- D20 pad 1: ROW1 -> Net-(D20-Pad1)
- D21 pad 1: ROW1 -> Net-(D21-Pad1)
- D22 pad 1: ROW1 -> Net-(D22-Pad1)
- D23 pad 1: ROW1 -> Net-(D23-Pad1)
- D24 pad 1: ROW1 -> Net-(D24-Pad1)
- D25 pad 1: ROW1 -> ROW2
- D26 pad 1: ROW1 -> Net-(D26-Pad1)
- D27 pad 1: ROW1 -> Net-(D27-Pad1)
- D28 pad 1: ROW1 -> Net-(D28-Pad1)
- D29 pad 1: ROW1 -> Net-(D29-Pad1)
- D30 pad 1: ROW1 -> Net-(D30-Pad1)
- D31 pad 1: ROW1 -> Net-(D31-Pad1)
- D32 pad 1: ROW1 -> Net-(D32-Pad1)
- D35 pad 1: ROW2 -> ROW4
- D36 pad 1: ROW2 -> ROW4
- D37 pad 1: ROW2 -> Net-(D37-Pad1)
- D4 pad 1: ROW0 -> Net-(D4-Pad1)
- D5 pad 1: ROW0 -> Net-(D5-Pad1)
- D6 pad 1: ROW0 -> Net-(D6-Pad1)
- D7 pad 1: ROW0 -> Net-(D7-Pad1)
- D8 pad 1: ROW0 -> Net-(D8-Pad1)
- D9 pad 1: ROW0 -> Net-(D9-Pad1)
- MX10 pad 2: Net-(D12-Pad2) -> Net-(D8-Pad1)
- MX11 pad 2: Net-(D13-Pad2) -> Net-(D8-Pad2)
- MX12 pad 2: Net-(D14-Pad2) -> Net-(D9-Pad1)
- MX13 pad 2: Net-(D15-Pad2) -> Net-(D9-Pad2)
- MX14 pad 2: Net-(D16-Pad2) -> Net-(D10-Pad1)
- MX15 pad 1: COL13 -> Net-(D10-Pad1)
- MX15 pad 2: Net-(D16-Pad2) -> COL13
- MX16 pad 2: Net-(D18-Pad2) (its old number) -> Net-(D10-Pad2)
- MX17 pad 2: Net-(D19-Pad2) -> Net-(D11-Pad2)
- MX18 pad 2: Net-(D20-Pad2) -> Net-(D11-Pad1)
- MX19 pad 2: Net-(D21-Pad2) -> Net-(D12-Pad2)
- MX2 pad 2: Net-(D4-Pad2) -> Net-(D4-Pad1)
- MX20 pad 2: Net-(D22-Pad2) -> Net-(D12-Pad1)
- MX21 pad 2: Net-(D23-Pad2) -> Net-(D13-Pad2)
- MX22 pad 2: Net-(D24-Pad2) -> Net-(D13-Pad1)
- MX23 pad 2: Net-(D25-Pad2) -> Net-(D14-Pad2)
- MX24 pad 2: Net-(D26-Pad2) -> Net-(D14-Pad1)
- MX25 pad 2: Net-(D27-Pad2) -> Net-(D15-Pad2)
- MX26 pad 2: Net-(D28-Pad2) -> Net-(D15-Pad1)
- MX27 pad 2: Net-(D29-Pad2) -> Net-(D16-Pad2)
- MX28 pad 2: Net-(D30-Pad2) -> Net-(D16-Pad1)
- MX29 pad 2: Net-(D31-Pad2) -> Net-(D17-Pad2)
- MX3 pad 2: Net-(D5-Pad2) -> Net-(D4-Pad2)
- MX30 pad 2: Net-(D32-Pad2) -> Net-(D17-Pad1)
- MX33 pad 2: Net-(D35-Pad2) -> Net-(D19-Pad1)
- MX34 pad 2: Net-(D36-Pad2) -> Net-(D19-Pad2)
- MX35 pad 2: Net-(D37-Pad2) -> Net-(D20-Pad1)
- MX36 pad 2: Net-(D38-Pad2) -> Net-(D20-Pad2)
- MX37 pad 2: Net-(D39-Pad2) -> Net-(D21-Pad1)
- MX38 pad 2: Net-(D40-Pad2) -> Net-(D21-Pad2)
- MX39 pad 2: Net-(D41-Pad2) -> Net-(D22-Pad1)
- MX4 pad 2: Net-(D6-Pad2) -> Net-(D5-Pad1)
- MX40 pad 2: Net-(D42-Pad2) -> Net-(D22-Pad2)
- MX41 pad 2: Net-(D43-Pad2) -> Net-(D23-Pad1)
- MX42 pad 2: Net-(D44-Pad2) -> Net-(D23-Pad2)
- MX43 pad 2: Net-(D45-Pad2) -> Net-(D24-Pad1)
- MX44 pad 2: Net-(D46-Pad2) -> Net-(D24-Pad2)
- MX45 pad 2: Net-(D47-Pad2) -> Net-(D25-Pad2)
- MX46 pad 2: Net-(D47-Pad2) -> Net-(D25-Pad2)
- MX47 pad 2: Net-(D49-Pad2) -> Net-(D26-Pad2)
- MX48 pad 2: Net-(D49-Pad2) -> Net-(D26-Pad2)
- MX49 pad 2: Net-(D51-Pad2) -> Net-(D26-Pad1)
- MX5 pad 2: Net-(D7-Pad2) -> Net-(D5-Pad2)
- MX50 pad 2: Net-(D52-Pad2) -> Net-(D27-Pad2)
- MX51 pad 2: Net-(D53-Pad2) -> Net-(D27-Pad1)
- MX52 pad 2: Net-(D54-Pad2) -> Net-(D28-Pad2)
- MX53 pad 2: Net-(D55-Pad2) -> Net-(D28-Pad1)
- MX54 pad 2: Net-(D56-Pad2) -> Net-(D29-Pad2)
- MX55 pad 2: Net-(D57-Pad2) -> Net-(D29-Pad1)
- MX56 pad 2: Net-(D58-Pad2) -> Net-(D30-Pad2)
- MX57 pad 2: Net-(D59-Pad2) -> Net-(D30-Pad1)
- MX58 pad 2: Net-(D60-Pad2) -> Net-(D31-Pad2)
- MX59 pad 2: Net-(D61-Pad2) -> Net-(D31-Pad1)
- MX6 pad 2: Net-(D8-Pad2) -> Net-(D6-Pad1)
- MX60 pad 2: Net-(D62-Pad2) -> Net-(D32-Pad2)
- MX61 pad 2: Net-(D62-Pad2) -> Net-(D32-Pad2)
- MX62 pad 2: Net-(D64-Pad2) -> Net-(D32-Pad1)
- MX66 pad 2: Net-(D68-Pad2) -> Net-(D35-Pad2)
- MX67 pad 2: Net-(D69-Pad2) -> Net-(D36-Pad2)
- MX68 pad 2: Net-(D70-Pad2) -> Net-(D37-Pad2)
- MX69 pad 2: Net-(D71-Pad2) -> Net-(D37-Pad1)
- MX7 pad 2: Net-(D9-Pad2) -> Net-(D6-Pad2)
- MX8 pad 2: Net-(D10-Pad2) -> Net-(D7-Pad1)
- MX9 pad 2: Net-(D11-Pad2) -> Net-(D7-Pad2)
Routing:
- net Net-(D47-Pad2): track 33.9 -> 0.00 mm
- net Net-(D23-Pad1): track 0.00 -> 27.4 mm, vias 0 -> 1
- net Net-(D18-Pad2) (its old number): track 26.7 -> 0.00 mm
- net Net-(D46-Pad2): track 24.5 -> 0.00 mm
- net Net-(D25-Pad2): track 12.0 -> 33.9 mm
- net Net-(D39-Pad2): track 20.5 -> 0.00 mm
- net Net-(D41-Pad2): track 20.4 -> 0.00 mm
- net Net-(D38-Pad2): track 20.1 -> 0.00 mm
- net Net-(D43-Pad2): track 19.8 -> 0.00 mm
- net Net-(D45-Pad2): track 19.7 -> 0.00 mm
- net ROW1: track 325.2 -> 306.3 mm, vias 4 -> 2
- net Net-(D32-Pad1): track 0.00 -> 17.4 mm
- net Net-(D4-Pad1): track 0.00 -> 16.5 mm
- net Net-(D5-Pad1): track 0.00 -> 16.5 mm
- net Net-(D7-Pad1): track 0.00 -> 16.4 mm
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
Commit message: rounding of traces
Routing:
- net COL5: track 208.4 -> 197.8 mm
- net COL7: track 153.8 -> 148.6 mm
- net COL14: track 220.1 -> 215.0 mm
- net COL3: track 240.1 -> 235.9 mm
- net COL6: track 181.2 -> 177.2 mm
- net COL9: track 141.6 -> 138.2 mm
- net VBUS: track 366.4 -> 369.4 mm
- net COL0: track 316.1 -> 319.1 mm
- net COL1: track 292.7 -> 289.9 mm
- net ROW2: track 291.1 -> 288.3 mm
- net COL13: track 215.9 -> 213.3 mm
- net USB-D+: track 256.9 -> 254.5 mm
- net USB-D-: track 257.6 -> 255.1 mm
- net Net-(D25-Pad2): track 33.9 -> 31.8 mm
- net COL11: track 205.0 -> 203.1 mm
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
Commit message: further beautification
Routing:
- net ROW2: track 288.3 -> 287.2 mm
- net Net-(D23-Pad1): track 28.3 -> 29.3 mm
- net ROW0: track 331.1 -> 330.2 mm
- net ROW3: track 267.8 -> 267.0 mm
- net ROW1: track 304.9 -> 304.3 mm
- net ROW4: track 249.5 -> 248.9 mm

Commit message: further changes
Routing:
- net Net-(D26-Pad1): track 11.9 -> 10.8 mm
- net Net-(D28-Pad1): track 9.79 -> 10.7 mm
- net Net-(D28-Pad2): track 9.62 -> 10.5 mm
- net Net-(D27-Pad2): track 9.62 -> 10.5 mm
- net Net-(D29-Pad2): track 9.62 -> 10.5 mm
- net Net-(D31-Pad1): track 9.73 -> 10.6 mm
- net Net-(D31-Pad2): track 9.56 -> 10.4 mm
- net Net-(D29-Pad1): track 9.79 -> 10.6 mm
- net Net-(D30-Pad2): track 9.62 -> 10.5 mm
- net Net-(D27-Pad1): track 9.73 -> 10.6 mm
- net Net-(D30-Pad1): track 9.79 -> 10.6 mm
- net Net-(D15-Pad2): track 9.17 -> 10.0 mm
- net Net-(D16-Pad2): track 9.17 -> 10.0 mm
- net Net-(D13-Pad1): track 10.2 -> 11.0 mm
- net Net-(D12-Pad2): track 9.17 -> 10.0 mm
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
Commit message: improved symmetry
Routing:
- net Net-(D37-Pad2): track 14.2 -> 16.8 mm
- net Net-(D37-Pad1): track 13.3 -> 15.7 mm

Commit message: discovered a way to copy and paste traces reliably
Routing:
- net COL11: track 203.1 -> 188.5 mm
- net COL14: track 215.0 -> 202.4 mm
- net Net-(D23-Pad1): track 29.3 -> 17.7 mm, vias 1 -> 2
- net COL7: track 148.6 -> 143.2 mm
- net COL13: track 213.3 -> 207.9 mm
- net COL5: track 197.8 -> 192.9 mm
- net COL1: track 289.8 -> 285.7 mm
- net COL6: track 177.2 -> 180.6 mm
- net COL8: track 113.1 -> 116.4 mm
- net COL9: track 138.3 -> 135.2 mm
- net COL3: track 235.9 -> 233.2 mm
- net COL4: track 205.0 -> 206.8 mm
- net COL2: track 258.8 -> 260.1 mm
- net ROW2: track 287.1 -> 286.4 mm
- net COL10: track 109.6 -> 109.0 mm
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