File: ptm-60nrf.sch (KiCad schematic (older format))
At the start: 20 parts, among them J1 USB_C_Receptacle_USB2.0, J2 BAT, J4 SWD, Q1 AO3407, U1 TP4054, U2 XC6220B331MR-G, U3 nRF52840_holyiot_18010, U4 SRV05-4, Y1 32.768Hz

Commit message: swapped reset button
Parts:
- Reset1: footprint Button_Switch_SMD:SW_SPST_B3U-1000P -> Button_Switch_SMD:SW_SPST_SKQG_WithStem
Changed lines of the file:
@@
 F 0 "Reset1" H 8600 2535 50  0000 C CNN
 F 1 "SW_Push" H 8600 2444 50  0000 C CNN
-F 2 "Button_Switch_SMD:SW_SPST_B3U-1000P" H 8600 2450 50  0001 C CNN
+F 2 "Button_Switch_SMD:SW_SPST_SKQG_WithStem" H 8600 2450 50  0001 C CNN
 F 3 "~" H 8600 2450 50  0001 C CNN
 	1    8600 2250

Commit message: minor fixes
Parts:
- removed Y1: 32.768Hz, Crystal:Crystal_SMD_MicroCrystal_CM9V-T1A-2Pin_1.6x1.0mm, symbol Device:Crystal_Small
- J4: footprint Connector_PinSocket_2.54mm:PinSocket_1x03_P2.54mm_Vertical -> Connector_PinSocket_2.54mm:PinSocket_1x04_P2.54mm_Vertical; symbol Connector_Generic:Conn_01x03 -> Connector_Generic:Conn_01x04
Connections:
- wire segments 58 -> 57
Changed lines of the file:
@@
 $EndComp
 Wire Wire Line
-	3700 4800 4550 4800
+	3700 4800 4250 4800
 Text GLabel 3400 6650 3    50   BiDi ~ 0
 USB-D-
@@
 	3300 6650 3300 6500
 $Comp
-L Connector_Generic:Conn_01x03 J4
+L Connector_Generic:Conn_01x04 J4
 U 1 1 60B2E742
-P 4450 5400
-F 0 "J4" H 4450 5700 50  0000 R CNN
-F 1 "SWD" H 4500 5600 50  0000 R CNN
-F 2 "Connector_PinSocket_2.54mm:PinSocket_1x03_P2.54mm_Vertical" H 4450 5400 50  0001 C CNN
-F 3 "~" H 4450 5400 50  0001 C CNN
-	1    4450 5400
+P 4450 5300
+F 0 "J4" H 4450 5600 50  0000 R CNN
+F 1 "SWD" H 4500 5500 50  0000 R CNN
+F 2 "Connector_PinSocket_2.54mm:PinSocket_1x04_P2.54mm_Vertical" H 4450 5300 50  0001 C CNN
+F 3 "~" H 4450 5300 50  0001 C CNN
+	1    4450 5300
 	1    0    0    -1
 $EndComp
@@
 Wire Wire Line
 	4250 6000 4250 6100
-Wire Wire Line
-	4250 6000 4250 5500
 $Comp
 L power:GND #PWR010
@@
 Wire Wire Line
 	2200 6000 2300 6000
-Text GLabel 3800 5900 2    50   Output ~ 0
+Text GLabel 3800 5700 2    50   Output ~ 0
 COL7
-Wire Wire Line
-	3800 5900 3700 5900
-Text GLabel 3800 5700 2    50   Output ~ 0
+Text GLabel 3800 5600 2    50   Output ~ 0
 COL8
 Wire Wire Line
@@
 Text Notes 5300 600  0    50   ~ 0
 USB-C Port
-$Comp
-L Device:Crystal_Small Y1
-U 1 1 61023DE6
-P 4150 5700
-F 0 "Y1" V 4100 5850 50  0000 L CNN
-F 1 "32.768Hz" V 4200 5850 50  0000 L CNN
-F 2 "Crystal:Crystal_SMD_MicroCrystal_CM9V-T1A-2Pin_1.6x1.0mm" H 4150 5700 50  0001 C CNN
-F 3 "~" H 4150 5700 50  0001 C CNN
-	1    4150 5700
-	0    1    1    0
-$EndComp
-Wire Wire Line
-	4150 5600 3700 5600
-Wire Wire Line
-	4150 5800 3700 5800
 Text GLabel 2500 6650 3    50   Output ~ 0
 VDD
@@
 Wire Wire Line
 	6900 1700 6900 2400
+Wire Wire Line
+	3800 5600 3700 5600
+Wire Wire Line
+	4250 5200 4250 4800
+Connection ~ 4250 4800
+Wire Wire Line
+	4250 4800 4550 4800
+Text GLabel 4250 5500 3    50   Input ~ 0
+VDD
 $EndSCHEMATC

Commit message: squashed bugs in schematic and rewired pwr/chrg
Connections:
- net VBUS: no longer D2.1 (K), Q1.2 (S), U2.1 (VIN), U2.3 (EN)
- new net: D2.1 (K), Q1.2 (S), U2.1 (VIN), U2.3 (EN)
- no-connect marks 0 -> 28
Changed lines of the file:
@@
 U 1 1 610594FA
 P 2650 950
-F 0 "Q1" H 2855 996 50  0000 L CNN
-F 1 "AO3407" H 2850 900 50  0000 L CNN
+F 0 "Q1" H 2850 950 50  0000 L CNN
+F 1 "AO3407" H 2850 850 50  0000 L CNN
 F 2 "Package_TO_SOT_SMD:SOT-23" H 2850 1050 50  0001 C CNN
 F 3 "~" H 2650 950 50  0001 C CNN
@@
 	1    0    0    -1
 $EndComp
-Wire Wire Line
-	2450 1350 2650 1350
 Wire Wire Line
 	2750 1350 2750 1250
@@
 Wire Wire Line
 	2650 1350 2750 1350
-Connection ~ 2650 1350
 $Comp
 L Regulator_Linear:AP2112K-3.3 U2
@@
 Wire Wire Line
 	4250 750  4700 750
-Text GLabel 4300 950  0    50   Input ~ 0
-VBAT
 $Comp
 L Device:R_Small R1
@@
 $EndComp
 $Comp
-L power:PWR_FLAG #FLG02
-U 1 1 610AA7ED
-P 8950 1000
-F 0 "#FLG02" H 8950 1075 50  0001 C CNN
-F 1 "PWR_FLAG" H 8950 1173 50  0000 C CNN
-F 2 "" H 8950 1000 50  0001 C CNN
-F 3 "~" H 8950 1000 50  0001 C CNN
-	1    8950 1000
-	1    0    0    -1
-$EndComp
-$Comp
-L power:PWR_FLAG #FLG03
-U 1 1 610AABBC
-P 9400 1000
-F 0 "#FLG03" H 9400 1075 50  0001 C CNN
-F 1 "PWR_FLAG" H 9400 1173 50  0000 C CNN
-F 2 "" H 9400 1000 50  0001 C CNN
-F 3 "~" H 9400 1000 50  0001 C CNN
-	1    9400 1000
-	1    0    0    -1
-$EndComp
-$Comp
 L power:PWR_FLAG #FLG04
 U 1 1 610AB96B
@@
 	1    0    0    -1
 $EndComp
-Text GLabel 8950 1000 3    50   Input ~ 0
-VDD
-Text GLabel 9400 1000 3    50   Input ~ 0
-VBAT
 Text GLabel 9850 1000 3    50   Input ~ 0
 VBUS
@@
 Text GLabel 4250 5500 3    50   Input ~ 0
 VDD
+NoConn ~ 5700 1700
+NoConn ~ 5800 1700
+NoConn ~ 2300 5200
+NoConn ~ 2300 5100
+NoConn ~ 2300 5000
+NoConn ~ 2300 4900
+NoConn ~ 2300 4600
+NoConn ~ 2300 4500
+NoConn ~ 2300 4400
+NoConn ~ 2300 4300
+NoConn ~ 2300 4200
+NoConn ~ 2300 4100
+NoConn ~ 2300 4000
+NoConn ~ 2300 3900
+NoConn ~ 2300 3800
+NoConn ~ 3700 3800
+NoConn ~ 3700 3900
+NoConn ~ 3700 4000
+NoConn ~ 3700 4100
+NoConn ~ 3700 4200
+NoConn ~ 3700 4300
+NoConn ~ 3700 4400
+NoConn ~ 3700 4500
+NoConn ~ 3700 4600
+NoConn ~ 3700 5800
+NoConn ~ 3700 5900
+NoConn ~ 4500 1900
+NoConn ~ 4300 1900
+Text GLabel 4300 950  0    50   Input ~ 0
+VBAT
 $EndSCHEMATC

Commit message: created branch 0.2 for alternate mcu location. Heavy cleanup
Connections:
- net COL0: now also U3.7 (P0.02); no longer U3.13 (P0.05)
- net COL1: now also U3.8 (P0.28); no longer U3.15 (P0.07)
- net COL10: now also U3.30 (P1.02); no longer U3.8 (P0.28)
- net COL11: now also U3.33 (P1.04); no longer U3.9 (P0.29)
- net COL12: now also U3.34 (P1.06); no longer U3.10 (P0.30)
- net COL13: now also U3.35 (P0.09); no longer U3.11 (P0.31)
- net COL14: now also U3.36 (P0.10); no longer U3.12 (P0.04)
- net COL2: now also U3.9 (P0.29); no longer U3.16 (P1.09)
- net COL3: now also U3.10 (P0.30); no longer U3.17 (P0.12)
- net COL4: now also U3.11 (P0.31); no longer U3.18 (P0.23)
- net COL5: now also U3.12 (P0.04); no longer U3.19 (P0.21)
- net COL6: now also U3.13 (P0.05); no longer U3.20 (P0.19)
- net COL7: now also U3.15 (P0.07); no longer U3.28 (P1.03)
- net COL8: now also U3.16 (P1.09); no longer U3.29 (P1.01)
- net COL9: now also U3.29 (P1.01); no longer U3.7 (P0.02)
- net ROW0: now also U3.20 (P0.19); no longer U3.36 (P0.10)
- net ROW1: now also U3.19 (P0.21); no longer U3.35 (P0.09)
- net ROW2: now also U3.18 (P0.23); no longer U3.34 (P1.06)
- net ROW3: now also U3.17 (P0.12); no longer U3.33 (P1.04)
- net ROW4: now also U3.28 (P1.03); no longer U3.30 (P1.02)
Changed lines of the file:
@@
 F1 "matrix.sch" 50
 $EndSheet
-Text GLabel 3800 4900 2    50   Input ~ 0
+Text GLabel 3100 6650 3    50   Input ~ 0
 ROW0
-Text GLabel 3800 5000 2    50   Input ~ 0
+Text GLabel 3000 6650 3    50   Input ~ 0
 ROW1
-Text GLabel 3800 5100 2    50   Input ~ 0
+Text GLabel 2900 6650 3    50   Input ~ 0
 ROW2
-Text GLabel 3800 5200 2    50   Input ~ 0
+Text GLabel 2800 6650 3    50   Input ~ 0
 ROW3
-Text GLabel 3800 5500 2    50   Input ~ 0
+Text GLabel 3800 5700 2    50   Input ~ 0
 ROW4
 Wire Wire Line
@@
 Wire Wire Line
 	3800 5500 3700 5500
-Text GLabel 3100 6650 3    50   Output ~ 0
+Text GLabel 2200 6000 0    50   Output ~ 0
 COL6
 Wire Wire Line
 	3100 6500 3100 6650
-Text GLabel 3000 6650 3    50   Output ~ 0
+Text GLabel 2200 5900 0    50   Output ~ 0
 COL5
 Wire Wire Line
 	3000 6500 3000 6650
-Text GLabel 2900 6650 3    50   Output ~ 0
+Text GLabel 2200 5800 0    50   Output ~ 0
 COL4
 Wire Wire Line
 	2900 6500 2900 6650
-Text GLabel 2800 6650 3    50   Output ~ 0
+Text GLabel 2200 5700 0    50   Output ~ 0
 COL3
 Wire Wire Line
 	2800 6500 2800 6650
+Text GLabel 2200 5600 0    50   Output ~ 0
+COL2
+Wire Wire Line
+	2700 6500 2700 6650
+Text GLabel 2200 5500 0    50   Output ~ 0
+COL1
+Wire Wire Line
+	2600 6500 2600 6650
+Text GLabel 2200 5400 0    50   Output ~ 0
+COL0
+Wire Wire Line
+	2200 6000 2300 6000
+Text GLabel 2600 6650 3    50   Output ~ 0
+COL7
 Text GLabel 2700 6650 3    50   Output ~ 0
-COL2
-Wire Wire Line
-	2700 6500 2700 6650
-Text GLabel 2600 6650 3    50   Output ~ 0
-COL1
-Wire Wire Line
-	2600 6500 2600 6650
-Text GLabel 2200 6000 0    50   Output ~ 0
-COL0
-Wire Wire Line
-	2200 6000 2300 6000
-Text GLabel 3800 5700 2    50   Output ~ 0
-COL7
+COL8
+Wire Wire Line
+	3800 5700 3700 5700
 Text GLabel 3800 5600 2    50   Output ~ 0
-COL8
-Wire Wire Line
-	3800 5700 3700 5700
-Text GLabel 2200 5400 0    50   Output ~ 0
 COL9
 Wire Wire Line
 	2200 5400 2300 5400
-Text GLabel 2200 5900 0    50   Output ~ 0
+Text GLabel 3800 4900 2    50   Output ~ 0
 COL14
 Wire Wire Line
 	2200 5900 2300 5900
-Text GLabel 2200 5800 0    50   Output ~ 0
+Text GLabel 3800 5000 2    50   Output ~ 0
 COL13
 Wire Wire Line
 	2200 5800 2300 5800
-Text GLabel 2200 5700 0    50   Output ~ 0
+Text GLabel 3800 5100 2    50   Output ~ 0
 COL12
 Wire Wire Line
 	2200 5700 2300 5700
-Text GLabel 2200 5600 0    50   Output ~ 0
+Text GLabel 3800 5200 2    50   Output ~ 0
 COL11
 Wire Wire Line
 	2200 5600 2300 5600
-Text GLabel 2200 5500 0    50   Output ~ 0
+Text GLabel 3800 5500 2    50   Output ~ 0
 COL10
 Wire Wire Line
@@
 	1    0    0    -1
 $EndComp
-Wire Wire Line
-	2750 1350 2750 1250
 Connection ~ 2450 1350
 $Comp
@@
 	1    0    0    -1
 $EndComp
-Connection ~ 2750 1350
 $Comp
 L power:GND #PWR07
@@
 Wire Wire Line
 	2750 1150 2750 1250
-Connection ~ 2750 1250
 Text GLabel 3350 1250 2    50   Input ~ 0
 VDD
@@
 Text GLabel 4300 950  0    50   Input ~ 0
 VBAT
+Wire Wire Line
+	2750 1250 2750 1350
+Connection ~ 2750 1250
+Connection ~ 2750 1350
 $EndSCHEMATC

Commit message: updated branch and ordered pcb prototype
Parts:
- C1: value 1µF -> 1nF; JLCPCB (none) -> C46653
- D1: JLCPCB (none) -> C84256
- D2: footprint Diode_SMD:D_SOD-123 -> Diode_SMD:D_SMA; JLCPCB (none) -> C2480
- J1: JLCPCB (none) -> C165948
- Q1: JLCPCB (none) -> C181093
- R1: JLCPCB (none) -> C21190
- R2: JLCPCB (none) -> C25804
- R3: JLCPCB (none) -> C25803
- R4, R5: JLCPCB (none) -> C23186
- R6: value 820K -> 1M; JLCPCB (none) -> C22935
- R7: JLCPCB (none) -> C22766
- Reset1: JLCPCB (none) -> C202424
- U1: JLCPCB (none) -> C32574
- U2: JLCPCB (none) -> C86534
- U4: JLCPCB (none) -> C85364
Changed lines of the file:
@@
 F 2 "Connector_USB:USB_C_Receptacle_HRO_TYPE-C-31-M-12" H 6450 1100 50  0001 C CNN
 F 3 "https://www.usb.org/sites/default/files/documents/usb_type-c.zip" H 6450 1100 50  0001 C CNN
+F 4 "C165948" V 6300 1100 50  0001 C CNN "JLCPCB"
 	1    6300 1100
 	0    1    1    0
@@
 F 2 "Resistor_SMD:R_0603_1608Metric" H 6600 1800 50  0001 C CNN
 F 3 "~" H 6600 1800 50  0001 C CNN
+F 4 "C23186" H 6600 1800 50  0001 C CNN "JLCPCB"
 	1    6600 1800
 	1    0    0    -1
@@
 F 2 "Resistor_SMD:R_0603_1608Metric" H 6700 1800 50  0001 C CNN
 F 3 "~" H 6700 1800 50  0001 C CNN
+F 4 "C23186" H 6700 1800 50  0001 C CNN "JLCPCB"
 	1    6700 1800
 	1    0    0    -1
@@
 F 2 "Package_TO_SOT_SMD:SOT-23" H 2850 1050 50  0001 C CNN
 F 3 "~" H 2650 950 50  0001 C CNN
+F 4 "C181093" H 2650 950 50  0001 C CNN "JLCPCB"
 	1    2650 950
 	1    0    0    -1
@@
 F 2 "Resistor_SMD:R_0603_1608Metric" H 2450 1450 50  0001 C CNN
 F 3 "~" H 2450 1450 50  0001 C CNN
+F 4 "" H 2450 1450 50  0001 C CNN "JLCPB"
+F 5 "C25803" H 2450 1450 50  0001 C CNN "JLCPCB"
 	1    2450 1450
 	1    0    0    -1
@@
 F 0 "D2" H 2550 1150 50  0000 C CNN
 F 1 "SS14" H 2500 1250 50  0000 C CNN
-F 2 "Diode_SMD:D_SOD-123" V 2550 1350 50  0001 C CNN
+F 2 "Diode_SMD:D_SMA" V 2550 1350 50  0001 C CNN
 F 3 "~" V 2550 1350 50  0001 C CNN
+F 4 "C2480" H 2550 1350 50  0001 C CNN "JLCPCB"
 	1    2550 1350
 	-1   0    0    1
@@
 F 2 "Package_TO_SOT_SMD:SOT-23-5" H 3050 1675 50  0001 C CNN
 F 3 "https://www.diodes.com/assets/Datasheets/AP2112.pdf" H 3050 1450 50  0001 C CNN
+F 4 "C86534" H 3050 1350 50  0001 C CNN "JLCPCB"
 	1    3050 1350
 	1    0    0    -1
@@
 F 2 "Package_TO_SOT_SMD:SOT-23-5" H 4750 800 50  0001 L CIN
 F 3 "http://ww1.microchip.com/downloads/en/DeviceDoc/20001984g.pdf" H 4550 1000 50  0001 C CNN
+F 4 "C32574" H 4700 1050 50  0001 C CNN "JLCPCB"
 	1    4700 1050
 	-1   0    0    -1
@@
 F 2 "Resistor_SMD:R_0603_1608Metric" H 4300 1250 50  0001 C CNN
 F 3 "~" H 4300 1250 50  0001 C CNN
+F 4 "C21190" H 4300 1250 50  0001 C CNN "JLCPCB"
 	1    4300 1250
 	-1   0    0    1
@@
 F 2 "LED_SMD:LED_0805_2012Metric" H 4050 1100 50  0001 C CNN
 F 3 "~" H 4050 1100 50  0001 C CNN
+F 4 "C84256" V 4050 1100 50  0001 C CNN "JLCPCB"
 	1    4050 1100
 	0    -1   -1   0
@@
 F 2 "Resistor_SMD:R_0603_1608Metric" H 5100 1250 50  0001 C CNN
 F 3 "~" H 5100 1250 50  0001 C CNN
+F 4 "C25804" H 5100 1250 50  0001 C CNN "JLCPCB"
 	1    5100 1250
 	-1   0    0    1
@@
 P 1700 5200
 F 0 "R6" H 1759 5246 50  0000 L CNN
-F 1 "820K" H 1759 5155 50  0000 L CNN
+F 1 "1M" H 1759 5155 50  0000 L CNN
 F 2 "Resistor_SMD:R_0603_1608Metric" H 1700 5200 50  0001 C CNN
 F 3 "~" H 1700 5200 50  0001 C CNN
+F 4 "C22935" H 1700 5200 50  0001 C CNN "JLCPCB"
 	1    1700 5200
 	1    0    0    -1
@@
 F 2 "Resistor_SMD:R_0603_1608Metric" H 1700 5400 50  0001 C CNN
 F 3 "~" H 1700 5400 50  0001 C CNN
+F 4 "C22766" H 1700 5400 50  0001 C CNN "JLCPCB"
 	1    1700 5400
 	1    0    0    -1
@@
 P 4800 750
 F 0 "C1" V 4750 650 50  0000 C CNN
-F 1 "1µF" V 4750 850 50  0000 C CNN
+F 1 "1nF" V 4750 850 50  0000 C CNN
 F 2 "Capacitor_SMD:C_0805_2012Metric" H 4800 750 50  0001 C CNN
 F 3 "~" H 4800 750 50  0001 C CNN
+F 4 "C46653" V 4800 750 50  0001 C CNN "JLCPCB"
 	1    4800 750
 	0    1    1    0
@@
 F 2 "Button_Switch_SMD:SW_SPST_SKQG_WithStem" H 8600 2450 50  0001 C CNN
 F 3 "~" H 8600 2450 50  0001 C CNN
+F 4 "C202424" H 8600 2250 50  0001 C CNN "JLCPCB"
 	1    8600 2250
 	1    0    0    -1
@@
 F 2 "Package_TO_SOT_SMD:SOT-23-6" H 5100 1950 50  0001 C CNN
 F 3 "http://www.onsemi.com/pub/Collateral/SRV05-4-D.PDF" H 4400 2400 50  0001 C CNN
+F 4 "C85364" V 4400 2400 50  0001 C CNN "JLCPCB"
 	1    4400 2400
 	0    1    1    0

Commit message: added footprint for rotary encoder on esc - renamed v0.4
Parts:
- C1: footprint Capacitor_SMD:C_0805_2012Metric -> Capacitor_SMD:C_0402_1005Metric; JLCPCB C46653 -> C1523
Connections:
- net ROTA: now reaches U3.2 (P1.11)
- net ROTB: now reaches U3.3 (P1.10)
- no-connect marks 28 -> 26
Changed lines of the file:
@@
 F 0 "C1" V 4750 650 50  0000 C CNN
 F 1 "1nF" V 4750 850 50  0000 C CNN
-F 2 "Capacitor_SMD:C_0805_2012Metric" H 4800 750 50  0001 C CNN
+F 2 "Capacitor_SMD:C_0402_1005Metric" H 4800 750 50  0001 C CNN
 F 3 "~" H 4800 750 50  0001 C CNN
-F 4 "C46653" V 4800 750 50  0001 C CNN "JLCPCB"
+F 4 "C1523" V 4800 750 50  0001 C CNN "JLCPCB"
 	1    4800 750
 	0    1    1    0
@@
 NoConn ~ 2300 5200
 NoConn ~ 2300 5100
-NoConn ~ 2300 5000
-NoConn ~ 2300 4900
 NoConn ~ 2300 4600
 NoConn ~ 2300 4500
@@
 Connection ~ 2750 1250
 Connection ~ 2750 1350
+Text GLabel 2300 4900 0    50   Input ~ 0
+ROTA
+Text GLabel 2300 5000 0    50   Input ~ 0
+ROTB
 $EndSCHEMATC

Commit message: added support for daughterboard (jst footprint)
Parts:
- added J3: Conn_01x04_Male, Connector_JST:JST_SH_BM04B-SRSS-TB_1x04-1MP_P1.00mm_Vertical, symbol Connector:Conn_01x04_Male
Connections:
- net GND: now also J3.1 (Pin_1)
- net USB-D+: now also J3.2 (Pin_2)
- net USB-D-: now also J3.3 (Pin_3)
- net VBUS: now also J3.4 (Pin_4)
Changed lines of the file:
@@
 	5400 1100 5400 2400
 Wire Wire Line
-	6200 1700 6200 2400
+	6200 1700 6200 2200
 Wire Wire Line
-	6400 1700 6400 2400
+	6400 1700 6400 2300
 Wire Wire Line
 	6900 1700 6900 2400
@@
 Text GLabel 2300 5000 0    50   Input ~ 0
 ROTB
+$Comp
+L Connector:Conn_01x04_Male J3
+U 1 1 60C51412
+P 7450 2200
+F 0 "J3" H 7422 2082 50  0000 R CNN
+F 1 "Conn_01x04_Male" H 7422 2173 50  0000 R CNN
+F 2 "Connector_JST:JST_SH_BM04B-SRSS-TB_1x04-1MP_P1.00mm_Vertical" H 7450 2200 50  0001 C CNN
+F 3 "~" H 7450 2200 50  0001 C CNN
+	1    7450 2200
+	-1   0    0    -1
+$EndComp
+Wire Wire Line
+	6900 2400 7250 2400
+Wire Wire Line
+	6400 2300 7250 2300
+Connection ~ 6400 2300
+Wire Wire Line
+	6400 2300 6400 2400
+Wire Wire Line
+	6200 2200 7250 2200
+Connection ~ 6200 2200
+Wire Wire Line
+	6200 2200 6200 2400
+$Comp
+L power:GND #PWR0105
+U 1 1 60C583E0
+P 7100 1950
+F 0 "#PWR0105" H 7100 1700 50  0001 C CNN
+F 1 "GND" H 7105 1777 50  0000 C CNN
+F 2 "" H 7100 1950 50  0001 C CNN
+F 3 "" H 7100 1950 50  0001 C CNN
+	1    7100 1950
+	1    0    0    -1
+$EndComp
+Wire Wire Line
+	7250 2100 7250 1950
+Wire Wire Line
+	7250 1950 7100 1950
 $EndSCHEMATC
